File: Keyboard V2.kicad_sch (KiCad schematic)
At the start: 233 parts, among them J1 USB_C_Receptacle_USB2.0_16P, J2 Conn_01x05_Pin, P1 SW_Push, SW1 ESC, SW10 F9, SW11 F10, SW12 F11, SW13 F12, SW14 PrntScrn, SW15 RotaryEncoder_Switch, SW16 Til, SW17 1, SW18 2, SW19 3, SW2 F1, SW20 4, SW21 5, SW22 6, SW23 7, SW24 8, SW25 9, SW26 0, SW27 Min, SW28 Plus, SW29 Bs, SW3 F2, SW30 Del, SW31 Tab, SW32 Q, SW33 W, SW34 E, SW35 R, SW36 T, SW37 Y, SW38 U, SW39 I, SW4 F3, SW40 O, SW41 P, SW42 LBrck, SW43 RBrck, SW44 BSlsh, SW45 Home, SW46 Caps, SW47 A, SW48 S, SW49 D, SW5 F4, SW50 F, SW51 G, SW52 H, SW53 J, SW54 K, SW55 L, SW56 Semi, SW57 Quot, SW58 Enter, SW59 End, SW6 F5, SW60 LShft, SW61 Z, SW62 X, SW63 C, SW64 V, SW65 B, SW66 N, SW67 M, SW68 Comma, SW69 Prd, SW7 F6, SW70 Slash, SW71 RShft, SW72 Up, SW73 LCtrl, SW74 Supr, SW75 Alt, SW76 Space, SW77 RAlt, SW78 Fn, SW79 Left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

Commit message: Update to wider pitch header
Parts:
- J2: footprint Connector_PinHeader_1.27mm:PinHeader_1x05_P1.27mm_Horizontal -> Connector_PinHeader_2.54mm:PinHeader_1x05_P2.54mm_Horizontal
Changed lines of the file:
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@@
 			)
 		)
-		(property "Footprint" "Connector_PinHeader_1.27mm:PinHeader_1x05_P1.27mm_Horizontal"
+		(property "Footprint" "Connector_PinHeader_2.54mm:PinHeader_1x05_P2.54mm_Horizontal"
 			(at 476.25 267.97 0)
 			(effects

Commit message: Fix Mux caps + Crystal Pinout
Properly wire Mux capacitors to 3v3a and gnd, remove the power flag. Switch to correct symbol for crystal
Parts:
- removed Y1: Crystal_GND23, Crystal:Crystal_SMD_Abracon_ABM8G-4Pin_3.2x2.5mm, symbol Device:Crystal_GND23
- added Y2: Crystal_GND24, Crystal:Crystal_SMD_Abracon_ABM8G-4Pin_3.2x2.5mm, symbol Device:Crystal_GND24
Connections:
- net +3V3A: now also AM0.24 (VCC), AM1.24 (VCC), AM2.24 (VCC), AM3.24 (VCC), AM4.24 (VCC), AM5.24 (VCC), C102.2, C103.2, C104.2, C105.2, C106.2, C7.2; no longer C102.1, C103.1, C104.1, C105.1, C106.1, C7.1
- net GND: now also C102.1, C103.1, C104.1, C105.1, C106.1, C7.1, Y2.2, Y2.4
- net at C16.1, R13.2: now also Y2.1
- net at C15.1, U3.G1 (PH0-OSC_IN): now also Y2.3
