File: _restore_backup_2026-08-05T10-35-34-378/Keyboard V2.kicad_sch (KiCad schematic)
At the start: 247 parts, among them J0 Conn_01x06_Pin, J1 Conn_01x05_Pin, J2 USB_C_Receptacle_USB2.0_16P, P1 SW_Push, SW1 ESC, SW10 F9, SW11 F10, SW12 F11, SW13 F12, SW14 PrntScrn, SW15 Til, SW16 1, SW17 2, SW18 3, SW19 4, SW2 F1, SW20 5, SW21 6, SW22 7, SW23 8, SW24 RotaryEncoder_Switch, SW25 9, SW26 0, SW27 Min, SW28 Plus, SW29 Bs, SW3 F2, SW30 Del, SW31 Tab, SW32 Q, SW33 W, SW34 E, SW35 R, SW36 T, SW37 Y, SW38 U, SW39 I, SW4 F3, SW40 O, SW41 P, SW42 LBrck, SW43 RBrck, SW44 BSlsh, SW45 Home, SW46 Caps, SW47 A, SW48 S, SW49 D, SW5 F4, SW50 F, SW51 G, SW52 H, SW53 J, SW54 K, SW55 L, SW56 Semi, SW57 Quot, SW58 Enter, SW59 End, SW6 F5, SW60 LShft, SW61 Z, SW62 X, SW63 C, SW64 V, SW65 B, SW66 N, SW67 M, SW68 Comma, SW69 Prd, SW7 F6, SW70 Slash, SW71 RShft, SW72 Up, SW73 LCtrl, SW74 Supr, SW75 Alt, SW76 Space, SW77 RAlt, SW78 Fn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

Commit message: updated stm32 config
Parts:
- removed C0: 5uF, symbol Device:C
- removed C100, C101, C99: 100pF, Capacitor_SMD:C_0402_1005Metric, symbol Device:C
- removed C121, C92, C93, C94, C95, C98: 100nF, Capacitor_SMD:C_0402_1005Metric, symbol Device:C
- removed C26, C39, C64, C77, C88: 100nF, Capacitor_SMD:C_0603_1608Metric, symbol Device:C
- removed C78, C89: 10uF, Capacitor_SMD:C_0805_2012Metric, symbol Device:C
- removed C90, C91: 30pF, Capacitor_SMD:C_0402_1005Metric, symbol Device:C
- removed C96, C97: 2.2uF, Capacitor_SMD:C_0402_1005Metric, symbol Device:C
- removed J0: Conn_01x06_Pin, BM06B-SRSS-TB:JST_BM06B-SRSS-TB_LF__SN_, symbol Connector:Conn_01x06_Pin
- removed J2: USB_C_Receptacle_USB2.0_16P, Connector_USB:USB_C_Receptacle_HRO_TYPE-C-31-M-12, symbol Connector:USB_C_Receptacle_USB2.0_16P
- removed R20, R21, R22: 100R, Resistor_SMD:R_0402_1005Metric, symbol Device:R
- removed U1: MCP1700T-3302E/MAY, DFN-S6_2x2MC_MCH, symbol 2026-08-06_20-43-36:MCP1700T-3302E_MAY
- removed U2: STM32F723IEK6, STM32F723IEK6:IC_STM32F723IEK6, symbol STM32F723IEK6:STM32F723IEK6
- removed U3: USBLC6-2P6, Package_TO_SOT_SMD:SOT-666, symbol Power_Protection:USBLC6-2P6
- removed Y1: Crystal_GND24, Crystal:Crystal_SMD_Abracon_ABM8G-4Pin_3.2x2.5mm, symbol Device:Crystal_GND24
- added C10, C12, C2, C3, C4, C5, C6: 100nF, Capacitor_SMD:C_0402_1005Metric, symbol Device:C
- added C11: 1uF, Capacitor_SMD:C_0402_1005Metric, symbol Device:C
- added C13, C8, C9: 2.2uF, Capacitor_SMD:C_0402_1005Metric, symbol Device:C
- added C15, C16: 30pF, Capacitor_SMD:C_0402_1005Metric, symbol Device:C
- added C17, C18: 10uF, Capacitor_SMD:C_0805_2012Metric, symbol Device:C
- added C34: 10nF, Capacitor_SMD:C_0402_1005Metric, symbol Device:C
- added C7: 100nF, Capacitor_SMD:C_0603_1608Metric, symbol Device:C
- added J1: USB_C_Receptacle_USB2.0_16P, Connector_USB:USB_C_Receptacle_HRO_TYPE-C-31-M-12, symbol Connector:USB_C_Receptacle_USB2.0_16P
- added U1: MCP1700T-3302E/MAY, Package_DFN_QFN:DFN-6-1EP_2x2mm_P0.65mm_EP1x1.6mm, symbol Regulator_Linear:MCP1700x-120xxMB
- added U2: USBLC6-2P6, Package_TO_SOT_SMD:SOT-666, symbol Power_Protection:USBLC6-2P6
- added U3: STM32F723IEK6, STM32F723IEK6:IC_STM32F723IEK6, symbol STM32F723IEK6:STM32F723IEK6
- added Y2: Crystal_GND24, Crystal:Crystal_SMD_Abracon_ABM8G-4Pin_3.2x2.5mm, symbol Device:Crystal_GND24
- C102, C103, C104: value 100pF -> 100nF; footprint Capacitor_SMD:C_0402_1005Metric -> Capacitor_SMD:C_0603_1608Metric
- C105, C106: footprint Capacitor_SMD:C_0402_1005Metric -> Capacitor_SMD:C_0603_1608Metric
- C107, C108, C119: value 100nF -> 100pF
- C109, C120: value 1uF -> 100pF
- C111: value 2.2uF -> 100nF
- C118: value 10nF -> 100pF
- C14: footprint Capacitor_SMD:C_0603_1608Metric -> Capacitor_SMD:C_0402_1005Metric
- R1: value 100ohm -> 3.00K
- R10, R11: value 100R -> 10K
- R12: value 1k -> 10K; footprint Resistor_SMD:R_0402_1005Metric -> Resistor_SMD:R_0603_1608Metric
- R13: value 1k -> 100ohm; footprint Resistor_SMD:R_0402_1005Metric -> Resistor_SMD:R_0603_1608Metric
- R14: value 22R -> 1k; footprint Resistor_SMD:R_0402_1005Metric -> Resistor_SMD:R_0603_1608Metric
- R15, R16: value 10K -> 1k
- R17: value 22R -> 100R
- R18: value 10K -> 100R; footprint Resistor_SMD:R_0603_1608Metric -> Resistor_SMD:R_0402_1005Metric
- R19: value 1k -> 100R; footprint Resistor_SMD:R_0603_1608Metric -> Resistor_SMD:R_0402_1005Metric
- R2: value 10K -> 5.1k
- R3: value 3.00K -> 5.1k
- R4: value 5.1k -> 10K
- R5: value 5.1k -> 100R; footprint Resistor_SMD:R_0603_1608Metric -> Resistor_SMD:R_0402_1005Metric
- R7, R8: value 100R -> 22R
- renumbered C63 to C100, C76 to C101, C2 to C19, C15 to C20, C27 to C21, C40 to C22, C52 to C23, C65 to C24, C79 to C25, C3 to C26, C16 to C27, C41 to C29, C53 to C30, C66 to C31, C80 to C32, C4 to C33, C29 to C35, C42 to C36, C54 to C37, C67 to C38, C81 to C39, C5 to C40, C17 to C41, C30 to C42, C55 to C44, C68 to C45, C82 to C46, C6 to C47, C18 to C48, C31 to C49, C44 to C50, C56 to C51, C69 to C52, C83 to C53, C7 to C54, C19 to C55, C32 to C56, C45 to C57, C57 to C58, C70 to C59, C84 to C60, C8 to C61, C20 to C62, C33 to C63, C46 to C64, C58 to C65, C71 to C66, C85 to C67, C9 to C68, C21 to C69, C34 to C70, C47 to C71, C59 to C72, C72 to C73, C86 to C74, C10 to C75, C22 to C76, C35 to C77, C48 to C78, C60 to C79, C73 to C80, C87 to C81, C11 to C82, C23 to C83, C36 to C84, C49 to C85, C61 to C86, C74 to C87, C12 to C89, C24 to C90, C37 to C91, C50 to C92, C62 to C93, C75 to C94, C13 to C96, C25 to C97, C38 to C98, C51 to C99, J1 to J2, SW24 to SW15, SW15 to SW16, SW16 to SW17, SW17 to SW18, SW18 to SW19, SW19 to SW20, SW20 to SW21, SW21 to SW22, SW22 to SW23, SW23 to SW24
Connections:
- net +3V3: now also C110.2, C111.1, C113.1, C115.2, C116.1, C14.1, R10.1, R11.2, R12.2, C18.1, C2.1, C3.2, C4.2, C5.2, C6.2, U1.3 (VO), U3.C1 (VBAT), U3.C5 (VDD1), U3.C6 (PDR_ON), U3.C7 (VDD1), U3.C8 (VDDSDMMC), U3.C9 (VDD1), U3.F3 (VDD1), U3.G13 (VDD1), U3.G3 (VDD1), U3.H13 (VDDUSB), U3.J12 (VDD2), U3.J13 (VDD2), U3.K4 (VDD2), U3.N10 (VDD2), U3.N8 (VDD2), U3.N9 (VDD2); no longer C105.2, C106.1, C107.1, C108.1, C110.1, C116.2, C119.1, R15.2, R16.1, R18.2
- net +3V3A: now also C102.2, C103.2, C104.2, C105.2, C106.2, C10.2, C11.2, C12.2, C7.2, U3.P1 (VREF+), U3.R1 (VDDA); no longer C1.2, C109.2, C113.2, C115.2, C120.2, C14.2
- net +5V: now also C17.1, J1.A4 (VBUS), J1.A9 (VBUS), J1.B4 (VBUS), J1.B9 (VBUS), U1.2 (VI), U2.5 (VBUS)
- net D+: now also R8.1, U2.4 (I/O2); no longer R14.1
- net D-: now also R7.1, U2.6 (I/O1); no longer R17.1
- net ENC_A: now also R16.2; no longer R12.2
- net ENC_B: now also R15.1; no longer R13.1
- net ENC_SW: now also R14.2; no longer R19.2
- net GND: now also C106.1, C107.1, C108.1, C110.1, C111.2, C113.2, C116.2, C118.1, C119.1, C14.2, R1.1, R2.2, R3.2, R4.1, C10.1, C11.1, C12.1, C13.1, C15.2, C16.2, C17.2, C18.2, C2.2, C3.1, C34.2, C4.1, C5.1, C6.1, C7.1, C8.1, C9.2, J1.A1 (GND), J1.A12 (GND), J1.B1 (GND), J1.B12 (GND), J1.SH (SHIELD), U1.1 (GND), U2.2 (GND), U3.D5 (VSS1), U3.D7 (VSS1), U3.D8 (VSS1), U3.D9 (VSS1), U3.F10 (VSS2), U3.F12 (VSS2), U3.F2 (VSS1), U3.F6 (VSS1), U3.F7 (VSS1), U3.F8 (VSS1), U3.F9 (VSS1), U3.G10 (VSS2), U3.G12 (VSS2), U3.G2 (VSS2), U3.G6 (VSS2), U3.G7 (VSS2), U3.G8 (VSS2), U3.G9 (VSS2), U3.H10 (VSS3), U3.H12 (VSS3), U3.H6 (VSS3), U3.H7 (VSS3), U3.H8 (VSS3), U3.H9 (VSS3), U3.J10 (VSS4), U3.J6 (VSS3), U3.J7 (VSS3), U3.J8 (VSS3), U3.J9 (VSS4), U3.K10 (VSS4), U3.K6 (VSS4), U3.K7 (VSS4), U3.K8 (VSS4), U3.K9 (VSS4), U3.L4 (BYPASS_REG), U3.M1 (VSSA), U3.M8 (VSS4), U3.M9 (VSS4), U3.N1 (VREF-), Y2.2 (G), Y2.4 (G); no longer C106.2, C107.2, C108.2, C110.2, C111.1, C113.1, C116.1, C118.2, C119.2, C14.1, R2.1, R3.1, R4.2, R5.2
- net MUX_0: now also R5.1; no longer R6.1
- net MUX_1: now also R6.1; no longer R7.1
- net MUX_3: now also R17.1; no longer R10.1
- net MUX_4: now also R18.1; no longer R8.1
- net MUX_5: now also R19.1; no longer R11.1
- net SELECT0: now also U3.R8 (PE7)
- net SELECT1: now also U3.R7 (PF14)
- net SELECT2: now also U3.R6 (PF11)
- net SELECT3: now also U3.R5 (PB0)
- net SWCLK: now also U3.A14 (PA14/JTCK-SWCLK)
- net SWDIO: now also U3.A15 (PA13/JTMS-SWDIO)
- net SWO: now also U3.A10 (PB3/JTDO/TRACESWO)
- net at R1.2: now also U3.J15 (OTG_HS_REXT)
- net at R10.2: now also R15.2, U3.G15 (PC7); no longer C103.2
- net at R13.2: now also C16.1, Y2.1; no longer R16.2
- net at R7.2: now also U3.C15 (PA11)
- net at R9.2: now also C109.2, U3.P3 (PA6); no longer C102.2
- net at R12.1: now also R14.1, C34.1, U3.N14 (PD11); no longer R15.1
- net at R6.2: now also C108.2, U3.R2 (PA3)
- net at P1.2: now also C1.2, U3.J1 (~{RST})
- net at R8.2: now also U3.B15 (PA12)
- net at R17.2: now also C118.2, U3.R3 (PA7)
- new net: R4.2, U3.D6 (BOOT0)
- new net: R13.1, U3.H1 (PH1-OSC_OUT)
- new net: C15.1, U3.G1 (PH0-OSC_IN), Y2.3
- new net: R11.1, R16.1, U3.H15 (PC6)
- new net: C107.2, R5.2, U3.P2 (PA2)
- new net: C119.2, R18.2, U3.P4 (PA5)
- new net: C120.2, R19.2, U3.R4 (PB1)
- new net: J1.A5 (CC1), R2.1
- new net: C13.2, U3.J14 (VDD12OTGHS)
- new net: C9.1, U3.M10 (VCAP_1)
- new net: J1.B5 (CC2), R3.1
- new net: J1.A7 (D-), J1.B7 (D-), U2.1 (I/O1)
- new net: J1.A6 (D+), J1.B6 (D+), U2.3 (I/O2)
- new net: C8.2, U3.F13 (VCAP_2)
- no-connect marks 142 -> 136
Other:
- moved on the sheet: FID1, FID2, FID3, J2, S1, S2, S3, S4
