File: _restore_backup_2026-08-06T15-55-17-821/Keyboard V2.kicad_pcb (KiCad board)
At the start: 4 copper layers, 317.8 x 142.5 mm, 239 parts, among them J1 Conn_01x05_Pin, J2 USB_C_Receptacle_USB2.0_16P, P1 SW_Push, SW1 ESC, SW10 F9, SW11 F10, SW12 F11, SW13 F12, SW14 PrntScrn, SW15 Til, SW16 1, SW17 2, SW18 3, SW19 4, SW2 F1, SW20 5, SW21 6, SW22 7, SW23 8, SW24 RotaryEncoder_Switch, SW25 9, SW26 0, SW27 Min, SW28 Plus, SW29 Bs, SW3 F2, SW30 Del, SW31 Tab, SW32 Q, SW33 W, SW34 E, SW35 R, SW36 T, SW37 Y, SW38 U, SW39 I, SW4 F3, SW40 O, SW41 P, SW42 LBrck, SW43 RBrck, SW44 BSlsh, SW45 Home, SW46 Caps, SW47 A, SW48 S, SW49 D, SW5 F4, SW50 F, SW51 G, SW52 H, SW53 J, SW54 K, SW55 L, SW56 Semi, SW57 Quot, SW58 Enter, SW59 End, SW6 F5, SW60 LShft, SW61 Z, SW62 X, SW63 C, SW64 V, SW65 B, SW66 N, SW67 M, SW68 Comma, SW69 Prd, SW7 F6, SW70 Slash, SW71 RShft, SW72 Up, SW73 LCtrl, SW74 Supr, SW75 Alt, SW76 Space, SW77 RAlt, SW78 Fn, SW79 Left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

Commit message: updated stm32 config
Parts:
- removed the C100 at (304.1, 31.1)
- removed the C101 at (308.8, 31.2)
- removed the C26 at (86.0, 106.5)
- removed the C39 at (163.8, 103.9)
- removed the C64 at (248.2, 103.4)
- removed the C77 at (320.2, 108.1)
- removed the C78 at (339.4, 17.9)
- removed C88: 100nF, Capacitor_SMD:C_0603_1608Metric
- removed the C89 at (338.9, 23.6)
- removed the C90 at (304.7, 18.7)
- removed the C91 at (301.0, 22.8)
- removed the C92 at (310.5, 15.2)
- removed the C93 at (311.6, 15.2)
- removed the C94 at (313.8, 15.2)
- removed C95: 100nF, Capacitor_SMD:C_0402_1005Metric
- removed the C96 at (317.1, 29.3)
- removed the C97 at (320.2, 18.7)
- removed the C98 at (306.2, 20.7)
- removed the C99 at (302.6, 31.1)
- removed the J2 at (331.4, 14.6)
- removed Y1: Crystal_GND24, Crystal:Crystal_SMD_Abracon_ABM8G-4Pin_3.2x2.5mm
- added C10: 100nF, Capacitor_SMD:C_0402_1005Metric, F.Cu at (306.5, 26.0)
- added C11: 1uF, Capacitor_SMD:C_0402_1005Metric, F.Cu at (305.4, 26.0)
- added C119: 100pF, Capacitor_SMD:C_0402_1005Metric, F.Cu at (309.1, 30.4)
- added C12: 100nF, Capacitor_SMD:C_0402_1005Metric, F.Cu at (304.2, 26.0)
- added C120: 100pF, Capacitor_SMD:C_0402_1005Metric, F.Cu at (310.4, 30.4)
- added C13: 2.2uF, Capacitor_SMD:C_0402_1005Metric, F.Cu at (320.2, 23.4)
- added C15: 30pF, Capacitor_SMD:C_0402_1005Metric, F.Cu at (304.7, 18.8)
- added C16: 30pF, Capacitor_SMD:C_0402_1005Metric, F.Cu at (301.0, 22.8)
- added C17: 10uF, Capacitor_SMD:C_0805_2012Metric, F.Cu at (339.3, 19.0)
- added C18: 10uF, Capacitor_SMD:C_0805_2012Metric, F.Cu at (339.3, 23.9)
- added C2: 100nF, Capacitor_SMD:C_0402_1005Metric, F.Cu at (310.9, 15.3)
- added C3: 100nF, Capacitor_SMD:C_0402_1005Metric, F.Cu at (311.9, 15.3)
- added C34: 10nF, Capacitor_SMD:C_0402_1005Metric, F.Cu at (319.0, 30.3)
- added C4: 100nF, Capacitor_SMD:C_0402_1005Metric, F.Cu at (314.0, 15.3)
- added C5: 100nF, Capacitor_SMD:C_0402_1005Metric, F.Cu at (320.2, 19.7)
- added C6: 100nF, Capacitor_SMD:C_0402_1005Metric, F.Cu at (306.2, 18.8)
- added C7: 100nF, Capacitor_SMD:C_0603_1608Metric, B.Cu at (95.9, 46.8)
- added C8: 2.2uF, Capacitor_SMD:C_0402_1005Metric, F.Cu at (320.2, 18.7)
- added C9: 2.2uF, Capacitor_SMD:C_0402_1005Metric, F.Cu at (317.0, 29.3)
- added J1: USB_C_Receptacle_USB2.0_16P, Connector_USB:USB_C_Receptacle_HRO_TYPE-C-31-M-12, F.Cu at (331.4, 14.6)
- added Y2: Crystal_GND24, Crystal:Crystal_SMD_Abracon_ABM8G-4Pin_3.2x2.5mm, F.Cu at (302.1, 20.1)
- C1: moved to F.Cu
- C102, C103, C104: value 100pF -> 100nF; footprint Capacitor_SMD:C_0402_1005Metric -> Capacitor_SMD:C_0603_1608Metric; moved to B.Cu
- C105, C106: footprint Capacitor_SMD:C_0402_1005Metric -> Capacitor_SMD:C_0603_1608Metric; moved to B.Cu
- C107, C108: value 100nF -> 100pF
- C109: value 1uF -> 100pF
- C111: value 2.2uF -> 100nF
- C118: value 10nF -> 100pF
- C14: footprint Capacitor_SMD:C_0603_1608Metric -> Capacitor_SMD:C_0402_1005Metric; moved to F.Cu
- R1: value 100ohm -> 3.00K
- R10, R11: value 100R -> 10K
- R12: value 1k -> 10K; footprint Resistor_SMD:R_0402_1005Metric -> Resistor_SMD:R_0603_1608Metric
- R13: value 1k -> 100ohm; footprint Resistor_SMD:R_0402_1005Metric -> Resistor_SMD:R_0603_1608Metric
- R14: value 22R -> 1k; footprint Resistor_SMD:R_0402_1005Metric -> Resistor_SMD:R_0603_1608Metric
- R15, R16: value 10K -> 1k
- R17: value 22R -> 100R
- R18: value 10K -> 100R; footprint Resistor_SMD:R_0603_1608Metric -> Resistor_SMD:R_0402_1005Metric
- R19: value 1k -> 100R; footprint Resistor_SMD:R_0603_1608Metric -> Resistor_SMD:R_0402_1005Metric
- R2: value 10K -> 5.1k
- R3: value 3.00K -> 5.1k
- R4: value 5.1k -> 10K
- R5: value 5.1k -> 100R; footprint Resistor_SMD:R_0603_1608Metric -> Resistor_SMD:R_0402_1005Metric
- R7, R8: value 100R -> 22R
- U1: footprint footprints:DFN-S6_2x2MC_MCH -> Package_DFN_QFN:DFN-6-1EP_2x2mm_P0.65mm_EP1x1.6mm
- U2: value STM32F723IEK6 -> USBLC6-2P6; footprint STM32F723IEK6:IC_STM32F723IEK6 -> Package_TO_SOT_SMD:SOT-666
- U3: value USBLC6-2P6 -> STM32F723IEK6; footprint Package_TO_SOT_SMD:SOT-666 -> STM32F723IEK6:IC_STM32F723IEK6
- moved C103 233.7 mm to (86.0, 106.5), turned to 90 degrees
- moved C1 201.6 mm to (295.8, 20.5), turned to -90 degrees
- moved C104 163.5 mm to (163.8, 103.9), turned to 180 degrees
- moved C106 100.4 mm to (248.2, 103.3), turned to 0 degrees
- moved C105 89.6 mm to (320.2, 108.1), turned to 90 degrees
- moved C14 84.4 mm to (320.2, 27.2), turned to 0 degrees
- moved C102 69.3 mm to (238.2, 47.0), turned to 90 degrees
- moved R5 28.1 mm to (303.6, 32.4), turned to 90 degrees
- moved R2 26.2 mm to (333.2, 21.4)
- moved R4 26.2 mm to (307.9, 14.8)
- moved R7 22.3 mm to (320.2, 17.6), turned to 180 degrees
- moved R8 20.1 mm to (320.2, 16.6), turned to 180 degrees
- moved R13 19.6 mm to (303.4, 22.6), turned to 180 degrees
- moved R17 19.3 mm to (307.8, 32.4), turned to 90 degrees
- moved R10 19.0 mm to (321.8, 21.0), turned to -90 degrees
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- renumbered C63 to C100, C76 to C101, C2 to C19, C15 to C20, C27 to C21, C40 to C22, C52 to C23, C65 to C24, C79 to C25, C3 to C26, C16 to C27, C41 to C29, C53 to C30, C66 to C31, C80 to C32, C4 to C33, C29 to C35, C42 to C36, C54 to C37, C67 to C38, C81 to C39, C5 to C40, C17 to C41, C30 to C42, C55 to C44, C68 to C45, C82 to C46, C6 to C47, C18 to C48, C31 to C49, C44 to C50, C56 to C51, C69 to C52, C83 to C53, C7 to C54, C19 to C55, C32 to C56, C45 to C57, C57 to C58, C70 to C59, C84 to C60, C8 to C61, C20 to C62, C33 to C63, C46 to C64, C58 to C65, C71 to C66, C85 to C67, C9 to C68, C21 to C69, C34 to C70, C47 to C71, C59 to C72, C72 to C73, C86 to C74, C10 to C75, C22 to C76, C35 to C77, C48 to C78, C60 to C79, C73 to C80, C87 to C81, C11 to C82, C23 to C83, C36 to C84, C49 to C85, C61 to C86, C74 to C87, C12 to C89, C24 to C90, C37 to C91, C50 to C92, C62 to C93, C75 to C94, C13 to C96, C25 to C97, C38 to C98, C51 to C99, J1 to J2, SW24 to SW15, SW15 to SW16, SW16 to SW17, SW17 to SW18, SW18 to SW19, SW19 to SW20, SW20 to SW21, SW21 to SW22, SW22 to SW23, SW23 to SW24
Connections:
- C1 pad 2: +3V3A -> Net-(U3C-~{RST})
- C102 pad 2: Net-(U2B-PA6) -> +3V3A
- C103 pad 2: Net-(U2B-PA7) -> +3V3A
- C104 pad 2: Net-(U2B-PB1) -> +3V3A
- C105 pad 2: +3V3 -> +3V3A
- C106 pad 1: +3V3 -> GND
- C106 pad 2: GND -> +3V3A
- C107 pad 1: +3V3 -> GND
- C107 pad 2: GND -> Net-(U3B-PA2)
- C108 pad 1: +3V3 -> GND
- C108 pad 2: GND -> Net-(U3B-PA3)
- C109 pad 2: +3V3A -> Net-(U3B-PA6)
- C110 pad 1: +3V3 -> GND
- C110 pad 2: GND -> +3V3
- C111 pad 1: GND -> +3V3
- C111 pad 2: Net-(U2A-VDD12OTGHS) -> GND
- C113 pad 1: GND -> +3V3
- C113 pad 2: +3V3A -> GND
- C115 pad 2: +3V3A -> +3V3
- C116 pad 1: GND -> +3V3
- C116 pad 2: +3V3 -> GND
- C118 pad 1: Net-(U2B-PD11) -> GND
- C118 pad 2: GND -> Net-(U3B-PA7)
- C14 pad 1: GND -> +3V3
- C14 pad 2: +3V3A -> GND
- P1 pad 2: Net-(U2C-~{RST}) -> Net-(U3C-~{RST})
- R1 pad 1: Net-(U2C-PH1-OSC_OUT) -> GND
- R1 pad 2: Net-(C91-Pad1) -> Net-(U3C-OTG_HS_REXT)
- R10 pad 1: MUX_3 -> +3V3
- R10 pad 2: Net-(U2B-PA7) -> Net-(U3B-PC7)
- R11 pad 1: MUX_5 -> Net-(U3B-PC6)
- R11 pad 2: Net-(U2B-PB1) -> +3V3
- R12 pad 1: Net-(U2B-PC6) -> Net-(U3B-PD11)
- R12 pad 2: ENC_A -> +3V3
- R13 pad 1: ENC_B -> Net-(U3C-PH1-OSC_OUT)
- R13 pad 2: Net-(U2B-PC7) -> Net-(C16-Pad1)
- R14 pad 1: D+ -> Net-(U3B-PD11)
- R14 pad 2: Net-(U2B-PA12) -> ENC_SW
- R15 pad 1: Net-(U2B-PC6) -> ENC_B
- R15 pad 2: +3V3 -> Net-(U3B-PC7)
- R16 pad 1: +3V3 -> Net-(U3B-PC6)
- R16 pad 2: Net-(U2B-PC7) -> ENC_A
- R17 pad 1: D- -> MUX_3
- R17 pad 2: Net-(U2B-PA11) -> Net-(U3B-PA7)
- R18 pad 1: Net-(U2B-PD11) -> MUX_4
- R18 pad 2: +3V3 -> Net-(U3B-PA5)
- R19 pad 1: Net-(U2B-PD11) -> MUX_5
- R19 pad 2: ENC_SW -> Net-(U3B-PB1)
- R2 pad 1: GND -> Net-(J1-CC1)
- R2 pad 2: Net-(U2C-BOOT0) -> GND
- R3 pad 1: GND -> Net-(J1-CC2)
- R3 pad 2: Net-(U2C-OTG_HS_REXT) -> GND
- R4 pad 1: Net-(J2-CC1) -> GND
- R4 pad 2: GND -> Net-(U3C-BOOT0)
- R5 pad 1: Net-(J2-CC2) -> MUX_0
- R5 pad 2: GND -> Net-(U3B-PA2)
- R6 pad 1: MUX_0 -> MUX_1
- R6 pad 2: Net-(U2B-PA2) -> Net-(U3B-PA3)
- R7 pad 1: MUX_1 -> D-
- R7 pad 2: Net-(U2B-PA3) -> Net-(U3B-PA11)
- R8 pad 1: MUX_4 -> D+
- R8 pad 2: Net-(U2B-PA5) -> Net-(U3B-PA12)
- R9 pad 2: Net-(U2B-PA6) -> Net-(U3B-PA6)
- U1 pad 1: +5V -> GND
- U1 pad 2: unconnected-(U1-NC-Pad2) -> +5V
- U1 pad 3: GND -> +3V3
- U1 pad 4: unconnected-(U1-NC-Pad4) -> (no net)
- U1 pad 5: unconnected-(U1-NC-Pad5) -> (no net)
- U1 pad 6: +3V3 -> (no net)
- U1 pad 7: GND -> (no net)
Routing:
- net Net-(U2C-~{RST}): track 23.6 -> 0.00 mm, vias 2 -> 0
- net Net-(U3C-~{RST}): track 0.00 -> 23.3 mm, vias 0 -> 2
- net +3V3: track 110.3 -> 92.2 mm, vias 22 -> 27
- net Net-(U2B-PA2): track 11.5 -> 0.00 mm
- net Net-(U3B-PA2): track 0.00 -> 10.1 mm
- net Net-(U2B-PA3): track 9.76 -> 0.00 mm
- net Net-(U2B-PA6): track 9.46 -> 0.00 mm
- net Net-(U3B-PA6): track 0.00 -> 8.08 mm
- net Net-(U3B-PA3): track 0.00 -> 8.03 mm
- net Net-(U2C-PH0-OSC_IN): track 7.81 -> 0.00 mm
- net Net-(U2B-PA7): track 7.75 -> 0.00 mm
- net Net-(U3C-PH0-OSC_IN): track 0.00 -> 7.30 mm
- net Net-(U2B-PA5): track 7.26 -> 0.00 mm
- net Net-(U2C-BOOT0): track 6.80 -> 0.00 mm
- net Net-(U3C-BOOT0): track 0.00 -> 6.78 mm
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Other:
- board text removed: "AM0_0"
- board text removed: "AM0_1"
- board text removed: "AM0_10"
- board text removed: "AM0_11"
- board text removed: "AM0_12"
- board text removed: "AM0_13"
- board text removed: "AM0_14"
- board text removed: "AM0_15"
- board text removed: "AM0_2"
- board text removed: "AM0_3"
- board text removed: "AM0_4"
- board text removed: "AM0_5"
- board text removed: "AM0_6"
- board text removed: "AM0_9"
- board text removed: "AM1_0"
- board text removed: "AM1_1"
- board text removed: "AM1_10"
- board text removed: "AM1_11"
- board text removed: "AM1_12"
- board text removed: "AM1_13"
- board text removed: "AM1_14"
- board text removed: "AM1_15"
- board text removed: "AM1_2"
- board text removed: "AM1_3"
- board text removed: "AM1_4"
- board text removed: "AM1_5"
- board text removed: "AM1_7"
- board text removed: "AM1_9"
- board text removed: "AM2_0"
- board text removed: "AM2_1"
- board text removed: "AM2_10"
- board text removed: "AM2_11"
- board text removed: "AM2_12"
- board text removed: "AM2_13"
- board text removed: "AM2_14"
- board text removed: "AM2_15"
- board text removed: "AM2_2"
- board text removed: "AM2_3"
- board text removed: "AM2_4"
- board text removed: "AM2_5"
- board text removed: "AM2_6"
- board text removed: "AM2_8"
- board text removed: "AM2_9"
- board text removed: "AM3_0"
- board text removed: "AM3_1"
- board text removed: "AM3_10"
- board text removed: "AM3_11"
- board text removed: "AM3_12"
- board text removed: "AM3_13"
- board text removed: "AM3_14"
- board text removed: "AM3_15"
- board text removed: "AM3_2"
- board text removed: "AM3_3"
- board text removed: "AM3_4"
- board text removed: "AM3_5"
- board text removed: "AM3_6"
- board text removed: "AM3_7"
- board text removed: "AM3_8"
- board text removed: "AM3_9"
- board text removed: "AM4_1"
- board text removed: "AM4_10"
- board text removed: "AM4_11"
- board text removed: "AM4_12"
- board text removed: "AM4_13"
- board text removed: "AM4_14"
- board text removed: "AM4_2"
- board text removed: "AM4_3"
- board text removed: "AM4_4"
- board text removed: "AM4_5"
- board text removed: "AM4_6"
- board text removed: "AM4_7"
- board text removed: "AM4_8"
- board text removed: "AM4_9"
- board text removed: "AM5_0"
- board text removed: "AM5_1"
- board text removed: "AM5_13"
- board text removed: "AM5_14"
- board text removed: "AM5_15"
- board text removed: "AM5_6"
- board text removed: "AM5_7"
